Commit message: fix: seedling edit (250505)

File: src/piper_description/urdf/piper_description.urdf (robot description, URDF)
Before this commit: robot piper_description, 10 links, 9 joints
Joints:
- joint joint2: origin xyz=0 0 0 rpy=1.5708 -0.10095 -3.1416 -> xyz=0 0 0 rpy=1.5708 -0.2019 -3.1416

File: src/piper_description/urdf/piper_description.xacro (robot description, xacro)
@@ -153,5 +153,5 @@
     <origin
       xyz="0 0 0"
-      rpy="1.5708 -0.10095 -3.1416" />
+      rpy="1.5708 -0.2019 -3.1416" />
     <parent
       link="link1" />
@@ -385,5 +385,5 @@
     <origin
       xyz="8.8259E-05 -0.091 0"
-      rpy="1.5708 1.5708 0" />
+      rpy="1.5708 0 0" />
     <parent
       link="link5" />
